Commit message: change the marker 'sustc' to 'sustc todo'

File: turtlebot3_description/urdf/turtlebot3_burger.gazebo.xacro (robot description, xacro)
@@ -5,8 +5,8 @@
   <gazebo>
     <plugin name="turtlebot3_burger_controller" filename="libgazebo_ros_diff_drive.so">
-      <commandTopic>robot2/cmd_vel</commandTopic>   <!--SUSTC-->
-      <odometryTopic>robot2/odom</odometryTopic>    <!--SUSTC-->
-      <odometryFrame>robot2_odom</odometryFrame>    <!--SUSTC-->
-      <robotBaseFrame>robot2_base_footprint</robotBaseFrame>    <!--SUSTC-->
+      <commandTopic>robot2/cmd_vel</commandTopic>   <!--SUSTC TODO-->
+      <odometryTopic>robot2/odom</odometryTopic>    <!--SUSTC TODO-->
+      <odometryFrame>robot2_odom</odometryFrame>    <!--SUSTC TODO-->
+      <robotBaseFrame>robot2_base_footprint</robotBaseFrame>    <!--SUSTC TODO-->
       <publishWheelTF>false</publishWheelTF>
       <publishWheelJointState>true</publishWheelJointState>
@@ -21,8 +21,8 @@
     </plugin>
   </gazebo>
-  <gazebo reference="robot2_base_link"> <!--SUSTC-->
+  <gazebo reference="robot2_base_link"> <!--SUSTC TODO-->
     <material>Gazebo/Grey</material>
   </gazebo>
-  <gazebo reference="robot2_wheel_left_link">   <!--SUSTC-->
+  <gazebo reference="robot2_wheel_left_link">   <!--SUSTC TODO-->
     <mu1>10</mu1>
     <mu2>10</mu2>
@@ -34,5 +34,5 @@
     <material>Gazebo/DarkGrey</material>
   </gazebo>
-  <gazebo reference="robot2_wheel_right_link">  <!--SUSTC-->
+  <gazebo reference="robot2_wheel_right_link">  <!--SUSTC TODO-->
     <mu1>10</mu1>
     <mu2>10</mu2>
@@ -44,5 +44,5 @@
     <material>Gazebo/DarkGrey</material>
   </gazebo>
-  <gazebo reference="robot2_caster_back_link">  <!--SUSTC-->
+  <gazebo reference="robot2_caster_back_link">  <!--SUSTC TODO-->
     <mu1>0.0</mu1>
     <mu2>0.0</mu2>
@@ -56,7 +56,7 @@
     <plugin name="imu_plugin" filename="libgazebo_ros_imu.so">
       <alwaysOn>true</alwaysOn>
-      <bodyName>robot2_imu_link</bodyName>  <!--SUSTC-->
-      <topicName>/robot2/imu</topicName>    <!--SUSTC-->
-      <serviceName>/robot2_imu_service</serviceName>    <!--SUSTC-->
+      <bodyName>robot2_imu_link</bodyName>  <!--SUSTC TODO-->
+      <topicName>/robot2/imu</topicName>    <!--SUSTC TODO-->
+      <serviceName>/robot2_imu_service</serviceName>    <!--SUSTC TODO-->
       <gaussianNoise>0.0</gaussianNoise>
       <updateRate>100.0</updateRate>
@@ -80,5 +80,5 @@
     </plugin>
   </gazebo>
-  <gazebo reference="robot2_imu_link">  <!--SUSTC-->
+  <gazebo reference="robot2_imu_link">  <!--SUSTC TODO-->
     <sensor type="imu" name="imu">
       <always_on>true</always_on>
@@ -88,5 +88,5 @@
     <material>Gazebo/Grey</material>
   </gazebo>
-  <gazebo reference="robot2_base_scan"> <!--SUSTC-->
+  <gazebo reference="robot2_base_scan"> <!--SUSTC TODO-->
     <material>Gazebo/DarkGrey</material>
     <sensor type="ray" name="lds_lfcd_sensor">
@@ -115,6 +115,6 @@
       </ray>
       <plugin name="gazebo_ros_lds_lfcd_controller" filename="libgazebo_ros_laser.so">
-        <topicName>/robot2/scan</topicName> <!--SUSTC-->
-        <frameName>robot2_base_scan</frameName> <!--SUSTC-->
+        <topicName>/robot2/scan</topicName> <!--SUSTC TODO-->
+        <frameName>robot2_base_scan</frameName> <!--SUSTC TODO-->
       </plugin>
     </sensor>

File: turtlebot3_description/urdf/turtlebot3_burger.urdf.xacro (robot description, xacro)
@@ -3,11 +3,11 @@
   <xacro:include filename="$(find turtlebot3_description)/urdf/common_properties.xacro"/>
   <xacro:include filename="$(find turtlebot3_description)/urdf/turtlebot3_burger.gazebo.xacro"/>
-  <link name="robot2_base_footprint"/>  <!--SUSTC-->
-  <joint name="base_joint" type="fixed">    <!--SUSTC-->
-    <parent link="robot2_base_footprint"/>  <!--SUSTC-->
-    <child link="robot2_base_link"/>    <!--SUSTC-->
+  <link name="robot2_base_footprint"/>  <!--SUSTC TODO-->
+  <joint name="base_joint" type="fixed">    <!--SUSTC TODO-->
+    <parent link="robot2_base_footprint"/>  <!--SUSTC TODO-->
+    <child link="robot2_base_link"/>    <!--SUSTC TODO-->
     <origin xyz="0.0 0.0 0.010" rpy="0 0 0"/>
   </joint>
-  <link name="robot2_base_link">    <!--SUSTC-->
+  <link name="robot2_base_link">    <!--SUSTC TODO-->
     <visual>
       <origin xyz="-0.032 0 0.0" rpy="0 0 0"/>
@@ -32,10 +32,10 @@
   </link>
   <joint name="wheel_left_joint" type="continuous">
-    <parent link="robot2_base_link"/>   <!--SUSTC-->
-    <child link="robot2_wheel_left_link"/>  <!--SUSTC-->
+    <parent link="robot2_base_link"/>   <!--SUSTC TODO-->
+    <child link="robot2_wheel_left_link"/>  <!--SUSTC TODO-->
     <origin xyz="0.0 0.08 0.023" rpy="${-M_PI*0.5} 0 0"/>
     <axis xyz="0 0 1"/>
   </joint>
-  <link name="robot2_wheel_left_link">  <!--SUSTC-->
+  <link name="robot2_wheel_left_link">  <!--SUSTC TODO-->
     <visual>
       <origin xyz="0 0 0" rpy="${M_PI*0.5} 0 0"/>
@@ -60,10 +60,10 @@
   </link>
   <joint name="wheel_right_joint" type="continuous">
-    <parent link="robot2_base_link"/>   <!--SUSTC-->
-    <child link="robot2_wheel_right_link"/> <!--SUSTC-->
+    <parent link="robot2_base_link"/>   <!--SUSTC TODO-->
+    <child link="robot2_wheel_right_link"/> <!--SUSTC TODO-->
     <origin xyz="0.0 -0.08 0.023" rpy="${-M_PI*0.5} 0 0"/>
     <axis xyz="0 0 1"/>
   </joint>
-  <link name="robot2_wheel_right_link"> <!--SUSTC-->
+  <link name="robot2_wheel_right_link"> <!--SUSTC TODO-->
     <visual>
       <origin xyz="0 0 0" rpy="${M_PI*0.5} 0 0"/>
@@ -88,9 +88,9 @@
   </link>
   <joint name="caster_back_joint" type="fixed">
-    <parent link="robot2_base_link"/>   <!--SUSTC-->
-    <child link="robot2_caster_back_link"/> <!--SUSTC-->
+    <parent link="robot2_base_link"/>   <!--SUSTC TODO-->
+    <child link="robot2_caster_back_link"/> <!--SUSTC TODO-->
     <origin xyz="-0.081 0 -0.004" rpy="${-M_PI*0.5} 0 0"/>
   </joint>
-  <link name="robot2_caster_back_link"> <!--SUSTC-->
+  <link name="robot2_caster_back_link"> <!--SUSTC TODO-->
     <collision>
       <origin xyz="0 0 0" rpy="0 0 0"/>
@@ -108,15 +108,15 @@
   </link>
   <joint name="imu_joint" type="fixed">
-    <parent link="robot2_base_link"/>   <!--SUSTC-->
-    <child link="robot2_imu_link"/> <!--SUSTC-->
+    <parent link="robot2_base_link"/>   <!--SUSTC TODO-->
+    <child link="robot2_imu_link"/> <!--SUSTC TODO-->
     <origin xyz="-0.032 0 0.068" rpy="0 0 0"/>
   </joint>
-  <link name="robot2_imu_link"/>    <!--SUSTC-->
+  <link name="robot2_imu_link"/>    <!--SUSTC TODO-->
   <joint name="scan_joint" type="fixed">
-    <parent link="robot2_base_link"/>   <!--SUSTC-->
-    <child link="robot2_base_scan"/>    <!--SUSTC-->
+    <parent link="robot2_base_link"/>   <!--SUSTC TODO-->
+    <child link="robot2_base_scan"/>    <!--SUSTC TODO-->
     <origin xyz="-0.032 0 0.171" rpy="0 0 0"/>
   </joint>
-  <link name="robot2_base_scan">    <!--SUSTC-->
+  <link name="robot2_base_scan">    <!--SUSTC TODO-->
     <visual>
       <origin xyz="0 0 0.0" rpy="0 0 0"/>
